Commit message: ros2 throuble

File: install/custom_robot_description/share/custom_robot_description/urdf/custom_cobot.urdf.xacro (robot description, xacro)
@@ -89,3 +89,157 @@
                         joint_name="link5__link6"
                         actuator_name="motor_link5__link6" />
+    <!-- ROS2 control tag -->
+    <!-- <ros2_control name="GazeboSimSystem" type="system" >
+        <hardware>
+            <plugin>gazebo_ros2_control/GazeboSystem</plugin>
+        </hardware>
+        <joint name="base_link__link1">
+            <command_interface name="position" />
+            <state_interface name="position" >
+                <param name="initial_value">0.0</param>
+            </state_interface>
+            <state_interface name="velocity" />
+        </joint>
+        <joint name="link1__link2">
+            <command_interface name="position" />
+            <state_interface name="position" >
+                <param name="initial_value">0.0</param>
+            </state_interface>
+            <state_interface name="velocity" />
+        </joint>
+        <joint name="link2__link3">
+            <command_interface name="position" />
+            <state_interface name="position" >
+                <param name="initial_value">0.0</param>
+            </state_interface>
+            <state_interface name="velocity" />
+        </joint>
+        <joint name="link3__link4">
+            <command_interface name="position" />
+            <state_interface name="position" >
+                <param name="initial_value">0.0</param>
+            </state_interface>
+            <state_interface name="velocity" />
+        </joint>
+        <joint name="link4__link5">
+            <command_interface name="position" />
+            <state_interface name="position" >
+                <param name="initial_value">0.0</param>
+            </state_interface>
+            <state_interface name="velocity" />
+        </joint>
+        <joint name="link5__link6">
+            <command_interface name="position" />
+            <state_interface name="position" >
+                <param name="initial_value">0.0</param>
+            </state_interface>
+            <state_interface name="velocity" />
+        </joint>
+        <joint name="link5__link6">
+            <command_interface name="position" />
+            <state_interface name="position" >
+                <param name="initial_value">0.0</param>
+            </state_interface>
+            <state_interface name="velocity" />
+        </joint>
+        <joint name="finger_right_joint">
+            <command_interface name="position" />
+            <state_interface name="position" >
+                <param name="initial_value">0.0</param>
+            </state_interface>
+            <state_interface name="velocity" />
+        </joint>
+        <joint name="finger_left_joint">
+            <param name="mimic">finger_right_joint</param>
+            <param name="multiplier">-1</param>
+            <command_interface name="position" />
+            <state_interface name="position" >
+                <param name="initial_value">0.0</param>
+            </state_interface>
+            <state_interface name="velocity" />
+        </joint>
+    </ros2_control> -->
+    <ros2_control name="GazeboSimSystem" type="system">
+        <hardware>
+            <plugin>
+                <plugin>gazebo_ros2_control/GazeboSystem</plugin>
+            </plugin>
+        </hardware>
+        <joint name="base_link__link1">
+            <command_interface name="position">
+                <param name="min">-6.28</param>
+                <param name="max">6.28</param>
+            </command_interface>
+            <state_interface name="position">
+                <param name="initial_value">0.0</param>
+            </state_interface>
+            <state_interface name="velocity" />
+        </joint>
+        <joint name="link1__link2">
+            <command_interface name="position">
+                <param name="min">-6.28</param>
+                <param name="max">6.28</param>
+            </command_interface>
+            <state_interface name="position" >
+                <param name="initial_value">0.0</param>
+            </state_interface>
+            <state_interface name="velocity" />
+        </joint>
+        <joint name="link2__link3">
+            <command_interface name="position">
+                <param name="min">-6.28</param>
+                <param name="max">6.28</param>
+            </command_interface>
+            <state_interface name="position" >
+                <param name="initial_value">0.0</param>
+            </state_interface>
+            <state_interface name="velocity" />
+        </joint>
+        <joint name="link3__link4">
+            <command_interface name="position">
+                <param name="min">-6.28</param>
+                <param name="max">6.28</param>
+            </command_interface>
+            <state_interface name="position" >
+                <param name="initial_value">0.0</param>
+            </state_interface>
+            <state_interface name="velocity" />
+        </joint>
+        <joint name="link4__link5">
+            <command_interface name="position">
+                <param name="min">-6.28</param>
+                <param name="max">6.28</param>
+            </command_interface>
+            <state_interface name="position" >
+                <param name="initial_value">0.0</param>
+            </state_interface>
+            <state_interface name="velocity" />
+        </joint>
+        <joint name="link5__link6">
+            <command_interface name="position">
+                <param name="min">-6.28</param>
+                <param name="max">6.28</param>
+            </command_interface>
+            <state_interface name="position" >
+                <param name="initial_value">0.0</param>
+            </state_interface>
+            <state_interface name="velocity" />
+        </joint>
+        <joint name="finger_right_joint">
+            <command_interface name="position" />
+            <state_interface name="position" >
+                <param name="initial_value">0.0</param>
+            </state_interface>
+            <state_interface name="velocity" />
+        </joint>
+        <joint name="finger_left_joint">
+            <param name="mimic">finger_right_joint</param>
+            <param name="multiplier">-1</param>
+            <command_interface name="position" />
+            <state_interface name="position" >
+                <param name="initial_value">0.0</param>
+            </state_interface>
+            <state_interface name="velocity" />
+        </joint>
+    </ros2_control>
 </robot>

File: install/custom_robot_description/share/custom_robot_description/urdf/custom_robot_gazebo.xacro (robot description, xacro)
@@ -1,8 +1,18 @@
 <?xml version = "1.0"?>
 <robot xmlns:xacro="http://www.ros.org/wiki/xacro">
-    <gazebo>
+    <!-- <gazebo>
         <plugin name="gazebo_ros_control" filename="libgazebo_ros_control.so">
             <robotNamespace>/cobot</robotNamespace>
-            <!-- <robotSimType>gazebo_ros_control/DefaultRobotHWSim</robotSimType> -->
+            <robotSimType>gazebo_ros_control/DefaultRobotHWSim</robotSimType>
+            <ros2_control>
+                <param name="robot_description">robot_description</param>
+            </ros2_control>
+        </plugin>
+    </gazebo> -->
+    <gazebo>
+        <plugin name="gazebo_ros2_control" filename = "libgazebo_ros2_control.so">
+            <parameters>$(find custom_robot_gazebo)/config/joint_controllers.yaml </parameters>
+            <!-- Namespace del robot -->
+            <robotNamespace>/cobot</robotNamespace>
         </plugin>
     </gazebo>

File: install/custom_robot_description/share/custom_robot_description/urdf/link_joint.xacro (robot description, xacro)
@@ -76,3 +76,34 @@
         </transmission>
     </xacro:macro>
+    <ros2_control name="CobotHardware" type="system">
+        <hardware>
+            <plugin>ros2_control_demo_hardware/CobotSystemEffortOnlyHardware</plugin>
+            <!-- Modifica il plugin con quello effettivo che utilizzi -->
+        </hardware>
+        <joint name="base_link__link1">
+            <state_interface name="effort"/>
+            <command_interface name="effort"/>
+        </joint>
+        <joint name="link1__link2">
+            <state_interface name="effort"/>
+            <command_interface name="effort"/>
+        </joint>
+        <joint name="link2__link3">
+            <state_interface name="effort"/>
+            <command_interface name="effort"/>
+        </joint>
+        <joint name="link3__link4">
+            <state_interface name="effort"/>
+            <command_interface name="effort"/>
+        </joint>
+        <joint name="link4__link5">
+            <state_interface name="effort"/>
+            <command_interface name="effort"/>
+        </joint>
+        <joint name="link5__link6">
+            <state_interface name="effort"/>
+            <command_interface name="effort"/>
+        </joint>
+        <!-- Aggiungi altri giunti con lo stesso formato -->
+    </ros2_control>
 </robot>
